Commit message: feat: Enhance vector_description package with new simulation and visualization capabilities, including IMU and LiDAR sensors, RViz configuration, and world definition for Gazebo.

File: src/vector_description/urdf/vector_urdf.xacro (robot description, xacro)
@@ -333,3 +333,19 @@
     <axis xyz="0.0 -1.0 0.0"/>
   </joint>
+  <!-- ============================================================ -->
+  <!-- IMU link — massless, centred on base (TurtleBot3 pattern)   -->
+  <!-- ============================================================ -->
+  <link name="imu_link">
+    <inertial>
+      <mass value="0.001"/>
+      <origin xyz="0 0 0" rpy="0 0 0"/>
+      <inertia ixx="1e-6" ixy="0" ixz="0" iyy="1e-6" iyz="0" izz="1e-6"/>
+    </inertial>
+  </link>
+  <!-- base_link → imu_link: mounted at robot centre, 20 mm above base plane -->
+  <joint name="imu_joint" type="fixed">
+    <origin xyz="0.0 0.0 0.02" rpy="0 0 0"/>
+    <parent link="base_link"/>
+    <child link="imu_link"/>
+  </joint>
 </robot>

Commit message: feat: Update launch files and URDF for improved sensor integration and performance in VECTOR NAV

File: src/vector_description/urdf/vector_urdf.xacro (robot description, xacro)
@@ -280,5 +280,5 @@
     <parent link="motor_rr"/>
     <child link="wheel_rr"/>
-    <axis xyz="0.0 -1.0 0.0"/>
+    <axis xyz="0.0 1.0 0.0"/>
   </joint>
   <!-- base_link → lidar_base (fixed) -->
@@ -331,5 +331,5 @@
     <parent link="motor_fr"/>
     <child link="wheel_fr"/>
-    <axis xyz="0.0 -1.0 0.0"/>
+    <axis xyz="0.0 1.0 0.0"/>
   </joint>
   <!-- ============================================================ -->

Commit message: fix: fixed the gazebo laggin by reducing the collision polygons

File: src/vector_description/urdf/vector_urdf.xacro (robot description, xacro)
@@ -60,7 +60,7 @@
     </visual>
     <collision>
-      <origin xyz="0 0 0" rpy="0 0 0"/>
-      <geometry>
-        <mesh filename="package://vector_description/meshes/base_link.stl" scale="0.001 0.001 0.001"/>
+      <origin xyz="0 0 0.015" rpy="0 0 0"/>
+      <geometry>
+        <box size="0.250 0.175 0.030"/>
       </geometry>
     </collision>
@@ -80,7 +80,7 @@
     </visual>
     <collision>
-      <origin xyz="0.063875 0.079 -0.0" rpy="0 0 0"/>
-      <geometry>
-        <mesh filename="package://vector_description/meshes/motor_rr.stl" scale="0.001 0.001 0.001"/>
+      <origin xyz="-0.008 0.017 -0.019" rpy="0 0 0"/>
+      <geometry>
+        <box size="0.029 0.070 0.033"/>
       </geometry>
     </collision>
@@ -100,7 +100,7 @@
     </visual>
     <collision>
-      <origin xyz="0.071875 0.089 0.019875" rpy="0 0 0"/>
-      <geometry>
-        <mesh filename="package://vector_description/meshes/wheel_rr.stl" scale="0.001 0.001 0.001"/>
+      <origin xyz="0.0 -0.018 0.0" rpy="1.5708 0 0"/>
+      <geometry>
+        <cylinder radius="0.034" length="0.032"/>
       </geometry>
     </collision>
@@ -120,7 +120,7 @@
     </visual>
     <collision>
-      <origin xyz="-0.05 0.02 -0.025" rpy="0 0 0"/>
-      <geometry>
-        <mesh filename="package://vector_description/meshes/lidar_base.stl" scale="0.001 0.001 0.001"/>
+      <origin xyz="0.024 0.020 0.035" rpy="0 0 0"/>
+      <geometry>
+        <box size="0.098 0.072 0.051"/>
       </geometry>
     </collision>
@@ -140,7 +140,7 @@
     </visual>
     <collision>
-      <origin xyz="-0.092 -0.0 -0.0732" rpy="0 0 0"/>
-      <geometry>
-        <mesh filename="package://vector_description/meshes/lidar_link.stl" scale="0.001 0.001 0.001"/>
+      <origin xyz="0.002 0.0 0.007" rpy="0 0 0"/>
+      <geometry>
+        <cylinder radius="0.035" length="0.030"/>
       </geometry>
     </collision>
@@ -160,7 +160,7 @@
     </visual>
     <collision>
-      <origin xyz="-0.079875 -0.079 -0.0" rpy="0 0 0"/>
-      <geometry>
-        <mesh filename="package://vector_description/meshes/motor_fl.stl" scale="0.001 0.001 0.001"/>
+      <origin xyz="-0.008 -0.017 -0.019" rpy="0 0 0"/>
+      <geometry>
+        <box size="0.029 0.070 0.033"/>
       </geometry>
     </collision>
@@ -180,7 +180,7 @@
     </visual>
     <collision>
-      <origin xyz="0.063825 -0.064 -0.0" rpy="0 0 0"/>
-      <geometry>
-        <mesh filename="package://vector_description/meshes/motor_rl.stl" scale="0.001 0.001 0.001"/>
+      <origin xyz="-0.008 -0.002 -0.019" rpy="0 0 0"/>
+      <geometry>
+        <box size="0.029 0.070 0.033"/>
       </geometry>
     </collision>
@@ -200,7 +200,7 @@
     </visual>
     <collision>
-      <origin xyz="-0.079825 0.064 -0.0" rpy="0 0 0"/>
-      <geometry>
-        <mesh filename="package://vector_description/meshes/motor_fr.stl" scale="0.001 0.001 0.001"/>
+      <origin xyz="-0.008 0.002 -0.019" rpy="0 0 0"/>
+      <geometry>
+        <box size="0.029 0.070 0.033"/>
       </geometry>
     </collision>
@@ -220,7 +220,7 @@
     </visual>
     <collision>
-      <origin xyz="-0.071875 -0.089 0.019875" rpy="0 0 0"/>
-      <geometry>
-        <mesh filename="package://vector_description/meshes/wheel_fl.stl" scale="0.001 0.001 0.001"/>
+      <origin xyz="0.0 0.018 0.0" rpy="1.5708 0 0"/>
+      <geometry>
+        <cylinder radius="0.034" length="0.032"/>
       </geometry>
     </collision>
@@ -240,7 +240,7 @@
     </visual>
     <collision>
-      <origin xyz="0.071776 -0.089 0.019875" rpy="0 0 0"/>
-      <geometry>
-        <mesh filename="package://vector_description/meshes/wheel_rl.stl" scale="0.001 0.001 0.001"/>
+      <origin xyz="0.0 0.018 0.0" rpy="1.5708 0 0"/>
+      <geometry>
+        <cylinder radius="0.034" length="0.032"/>
       </geometry>
     </collision>
@@ -260,7 +260,7 @@
     </visual>
     <collision>
-      <origin xyz="-0.071776 0.089 0.019875" rpy="0 0 0"/>
-      <geometry>
-        <mesh filename="package://vector_description/meshes/wheel_fr.stl" scale="0.001 0.001 0.001"/>
+      <origin xyz="0.0 -0.018 0.0" rpy="1.5708 0 0"/>
+      <geometry>
+        <cylinder radius="0.034" length="0.032"/>
       </geometry>
     </collision>
