Commit message: Update vector URDF materials, add teleoperation GUI package
- Changed materials for various components in vector_urdf.xacro from "silver" to more appropriate colors such as "dark_green", "dark_grey", "rubber_black", and "gunmetal".
- Updated vector_world.sdf to enable the sensors system plugin for GPU lidar and camera sensors.
- Introduced a new teleoperation GUI package (vector_teleop) with a Qt-based interface for controlling VECTOR NAV.
- Added launch file for teleoperation GUI.
- Created package.xml and setup.py for the new teleoperation package.
- Implemented the main teleoperation GUI logic in teleop_gui.py, including controls for movement and displaying odometry and IMU data.

File: src/vector_description/urdf/materials.xacro (robot description, xacro)
@@ -1,6 +1,19 @@
 <?xml version="1.0" ?>
 <robot name="vector_urdf" xmlns:xacro="http://www.ros.org/wiki/xacro" >
-<material name="silver">
-  <color rgba="0.700 0.700 0.700 1.000"/>
+<!-- Dark green metallic for base_link -->
+<material name="dark_green">
+  <color rgba="0.08 0.22 0.08 1.0"/>
+</material>
+<!-- Dark grey metallic for motors, lidar base -->
+<material name="dark_grey">
+  <color rgba="0.18 0.18 0.20 1.0"/>
+</material>
+<!-- Near-black rubber for wheels -->
+<material name="rubber_black">
+  <color rgba="0.05 0.05 0.05 1.0"/>
+</material>
+<!-- Gunmetal for lidar head -->
+<material name="gunmetal">
+  <color rgba="0.15 0.15 0.18 1.0"/>
 </material>
 </robot>

File: src/vector_description/urdf/vector_urdf.xacro (robot description, xacro)
@@ -57,5 +57,5 @@
         <mesh filename="package://vector_description/meshes/base_link.stl" scale="0.001 0.001 0.001"/>
       </geometry>
-      <material name="silver"/>
+      <material name="dark_green"/>
     </visual>
     <collision>
@@ -77,5 +77,5 @@
         <mesh filename="package://vector_description/meshes/motor_rr.stl" scale="0.001 0.001 0.001"/>
       </geometry>
-      <material name="silver"/>
+      <material name="dark_grey"/>
     </visual>
     <collision>
@@ -97,5 +97,5 @@
         <mesh filename="package://vector_description/meshes/wheel_rr.stl" scale="0.001 0.001 0.001"/>
       </geometry>
-      <material name="silver"/>
+      <material name="rubber_black"/>
     </visual>
     <collision>
@@ -117,5 +117,5 @@
         <mesh filename="package://vector_description/meshes/lidar_base.stl" scale="0.001 0.001 0.001"/>
       </geometry>
-      <material name="silver"/>
+      <material name="dark_grey"/>
     </visual>
     <collision>
@@ -137,5 +137,5 @@
         <mesh filename="package://vector_description/meshes/lidar_link.stl" scale="0.001 0.001 0.001"/>
       </geometry>
-      <material name="silver"/>
+      <material name="gunmetal"/>
     </visual>
     <collision>
@@ -157,5 +157,5 @@
         <mesh filename="package://vector_description/meshes/motor_fl.stl" scale="0.001 0.001 0.001"/>
       </geometry>
-      <material name="silver"/>
+      <material name="dark_grey"/>
     </visual>
     <collision>
@@ -177,5 +177,5 @@
         <mesh filename="package://vector_description/meshes/motor_rl.stl" scale="0.001 0.001 0.001"/>
       </geometry>
-      <material name="silver"/>
+      <material name="dark_grey"/>
     </visual>
     <collision>
@@ -197,5 +197,5 @@
         <mesh filename="package://vector_description/meshes/motor_fr.stl" scale="0.001 0.001 0.001"/>
       </geometry>
-      <material name="silver"/>
+      <material name="dark_grey"/>
     </visual>
     <collision>
@@ -217,5 +217,5 @@
         <mesh filename="package://vector_description/meshes/wheel_fl.stl" scale="0.001 0.001 0.001"/>
       </geometry>
-      <material name="silver"/>
+      <material name="rubber_black"/>
     </visual>
     <collision>
@@ -237,5 +237,5 @@
         <mesh filename="package://vector_description/meshes/wheel_rl.stl" scale="0.001 0.001 0.001"/>
       </geometry>
-      <material name="silver"/>
+      <material name="rubber_black"/>
     </visual>
     <collision>
@@ -257,5 +257,5 @@
         <mesh filename="package://vector_description/meshes/wheel_fr.stl" scale="0.001 0.001 0.001"/>
       </geometry>
-      <material name="silver"/>
+      <material name="rubber_black"/>
     </visual>
     <collision>
