Commit message: feat: Add vector_control package for RPi hardware control with Docker deployment
Implements ROS2 nodes for the Raspberry Pi 5 to control the VECTOR NAV robot hardware:
- Motor driver node: /cmd_vel subscription, diff-drive kinematics, feed-forward + PID
  velocity control with quadrature encoder feedback, publishes /wheel/odom
- IMU node: MPU6500 + HMC5883L reading with Madgwick AHRS filter, publishes /imu
- EKF config for real hardware fusing wheel odom + IMU gyro
- Docker setup (Dockerfile, docker-compose, systemd service) for RPi 5 with
  GPIO, I2C, camera, and CycloneDDS for Jetson-Pi communication
- Motor calibration tool for direction verification
- 25GA370 motors: 225 ticks/rev, LF encoder inverted, corrected pin mapping

Co-Authored-By: Claude Opus 4.6 <noreply@anthropic.com>

File: src/vector_ros/urdf/vector_urdf.xacro (robot description, xacro)
@@ -1,6 +1,6 @@
 <?xml version="1.0" ?>
 <robot name="vector_urdf" xmlns:xacro="http://www.ros.org/wiki/xacro">
-  <xacro:include filename="$(find vector_description)/urdf/materials.xacro" />
-  <xacro:include filename="$(find vector_description)/urdf/vector_urdf.gazebo" />
+  <xacro:include filename="$(find vector_ros)/urdf/materials.xacro" />
+  <xacro:include filename="$(find vector_ros)/urdf/vector_urdf.gazebo" />
   <!-- ============================================================ -->
   <!-- ros2_control hardware interface (velocity-controlled wheels) -->
@@ -55,5 +55,5 @@
       <origin xyz="0 0 0" rpy="0 0 0"/>
       <geometry>
-        <mesh filename="package://vector_description/meshes/base_link.stl" scale="0.001 0.001 0.001"/>
+        <mesh filename="package://vector_ros/meshes/base_link.stl" scale="0.001 0.001 0.001"/>
       </geometry>
       <material name="dark_green"/>
@@ -75,5 +75,5 @@
       <origin xyz="0.063875 0.079 -0.0" rpy="0 0 0"/>
       <geometry>
-        <mesh filename="package://vector_description/meshes/motor_rr.stl" scale="0.001 0.001 0.001"/>
+        <mesh filename="package://vector_ros/meshes/motor_rr.stl" scale="0.001 0.001 0.001"/>
       </geometry>
       <material name="dark_grey"/>
@@ -95,5 +95,5 @@
       <origin xyz="0.071875 0.089 0.019875" rpy="0 0 0"/>
       <geometry>
-        <mesh filename="package://vector_description/meshes/wheel_rr.stl" scale="0.001 0.001 0.001"/>
+        <mesh filename="package://vector_ros/meshes/wheel_rr.stl" scale="0.001 0.001 0.001"/>
       </geometry>
       <material name="rubber_black"/>
@@ -115,5 +115,5 @@
       <origin xyz="-0.05 0.02 -0.025" rpy="0 0 0"/>
       <geometry>
-        <mesh filename="package://vector_description/meshes/lidar_base.stl" scale="0.001 0.001 0.001"/>
+        <mesh filename="package://vector_ros/meshes/lidar_base.stl" scale="0.001 0.001 0.001"/>
       </geometry>
       <material name="dark_grey"/>
@@ -135,5 +135,5 @@
       <origin xyz="-0.092 -0.0 -0.0732" rpy="0 0 0"/>
       <geometry>
-        <mesh filename="package://vector_description/meshes/lidar_link.stl" scale="0.001 0.001 0.001"/>
+        <mesh filename="package://vector_ros/meshes/lidar_link.stl" scale="0.001 0.001 0.001"/>
       </geometry>
       <material name="gunmetal"/>
@@ -155,5 +155,5 @@
       <origin xyz="-0.079875 -0.079 -0.0" rpy="0 0 0"/>
       <geometry>
-        <mesh filename="package://vector_description/meshes/motor_fl.stl" scale="0.001 0.001 0.001"/>
+        <mesh filename="package://vector_ros/meshes/motor_fl.stl" scale="0.001 0.001 0.001"/>
       </geometry>
       <material name="dark_grey"/>
@@ -175,5 +175,5 @@
       <origin xyz="0.063825 -0.064 -0.0" rpy="0 0 0"/>
       <geometry>
-        <mesh filename="package://vector_description/meshes/motor_rl.stl" scale="0.001 0.001 0.001"/>
+        <mesh filename="package://vector_ros/meshes/motor_rl.stl" scale="0.001 0.001 0.001"/>
       </geometry>
       <material name="dark_grey"/>
@@ -195,5 +195,5 @@
       <origin xyz="-0.079825 0.064 -0.0" rpy="0 0 0"/>
       <geometry>
-        <mesh filename="package://vector_description/meshes/motor_fr.stl" scale="0.001 0.001 0.001"/>
+        <mesh filename="package://vector_ros/meshes/motor_fr.stl" scale="0.001 0.001 0.001"/>
       </geometry>
       <material name="dark_grey"/>
@@ -215,5 +215,5 @@
       <origin xyz="-0.071875 -0.089 0.019875" rpy="0 0 0"/>
       <geometry>
-        <mesh filename="package://vector_description/meshes/wheel_fl.stl" scale="0.001 0.001 0.001"/>
+        <mesh filename="package://vector_ros/meshes/wheel_fl.stl" scale="0.001 0.001 0.001"/>
       </geometry>
       <material name="rubber_black"/>
@@ -235,5 +235,5 @@
       <origin xyz="0.071776 -0.089 0.019875" rpy="0 0 0"/>
       <geometry>
-        <mesh filename="package://vector_description/meshes/wheel_rl.stl" scale="0.001 0.001 0.001"/>
+        <mesh filename="package://vector_ros/meshes/wheel_rl.stl" scale="0.001 0.001 0.001"/>
       </geometry>
       <material name="rubber_black"/>
@@ -255,5 +255,5 @@
       <origin xyz="-0.071776 0.089 0.019875" rpy="0 0 0"/>
       <geometry>
-        <mesh filename="package://vector_description/meshes/wheel_fr.stl" scale="0.001 0.001 0.001"/>
+        <mesh filename="package://vector_ros/meshes/wheel_fr.stl" scale="0.001 0.001 0.001"/>
       </geometry>
       <material name="rubber_black"/>
