Commit message: Update robot_info and configuration files for VECTOR NAV
- Updated language model in robot_info.txt from Qwen2.5-3B to Llama-3.2-3B-Instruct.
- Adjusted lidar_joint orientation in vector_urdf.xacro to correct the rotation.
- Added new EKF configuration file (ekf_hw.yaml) for real hardware integration.
- Created RViz configuration files (hw_nav.rviz and hw_slam.rviz) for navigation and SLAM visualization.
- Introduced nav2 parameters for hardware navigation (nav2_params_hw.yaml).
- Added SLAM Toolbox configuration for real hardware (slam_toolbox_hw.yaml).
- Implemented launch files for hardware navigation (hw_nav.launch.py) and SLAM (hw_slam.launch.py).

File: src/vector_ros/urdf/vector_urdf.xacro (robot description, xacro)
@@ -290,5 +290,5 @@
   <!-- lidar_base → lidar_link (fixed) -->
   <joint name="lidar_joint" type="fixed">
-    <origin xyz="0.042 0.02 0.0482" rpy="0 0 0"/>
+    <origin xyz="0.042 0.02 0.0482" rpy="0 0 3.14159"/>
     <parent link="lidar_base"/>
     <child link="lidar_link"/>
