Commit message: fix(nav): smooth navigation by removing motor brake and pinning min vels
Goal-driven motion was stuttering because the motor driver engaged an
active short-brake on every cmd_vel timeout, hard-locking the wheels
between bursts so each new cmd_vel had to fight the brake from a dead
stop. Coast at zero target instead — wheels keep their momentum
through brief gaps in the command stream.

Also align Nav2 controller and behavior min velocities with the Pi
motor driver hardware floor (linear 0.35 m/s, angular 2.25 rad/s) so
sub-floor commands are zeroed by the controller rather than snapped UP
by the motor driver into bang-bang kicks. Rename leftover vector_ros
package paths to vector_navigation in the hw_nav launch.

Co-Authored-By: Claude Opus 4.7 <noreply@anthropic.com>

File: src/vector_navigation/urdf/vector_urdf.xacro (robot description, xacro)
@@ -1,6 +1,6 @@
 <?xml version="1.0" ?>
 <robot name="vector_urdf" xmlns:xacro="http://www.ros.org/wiki/xacro">
-  <xacro:include filename="$(find vector_ros)/urdf/materials.xacro" />
-  <xacro:include filename="$(find vector_ros)/urdf/vector_urdf.gazebo" />
+  <xacro:include filename="$(find vector_navigation)/urdf/materials.xacro" />
+  <xacro:include filename="$(find vector_navigation)/urdf/vector_urdf.gazebo" />
   <!-- ============================================================ -->
   <!-- ros2_control hardware interface (velocity-controlled wheels) -->
@@ -55,5 +55,5 @@
       <origin xyz="0 0 0" rpy="0 0 0"/>
       <geometry>
-        <mesh filename="package://vector_ros/meshes/base_link.stl" scale="0.001 0.001 0.001"/>
+        <mesh filename="package://vector_navigation/meshes/base_link.stl" scale="0.001 0.001 0.001"/>
       </geometry>
       <material name="dark_green"/>
@@ -75,5 +75,5 @@
       <origin xyz="0.063875 0.079 -0.0" rpy="0 0 0"/>
       <geometry>
-        <mesh filename="package://vector_ros/meshes/motor_rr.stl" scale="0.001 0.001 0.001"/>
+        <mesh filename="package://vector_navigation/meshes/motor_rr.stl" scale="0.001 0.001 0.001"/>
       </geometry>
       <material name="dark_grey"/>
@@ -95,5 +95,5 @@
       <origin xyz="0.071875 0.089 0.019875" rpy="0 0 0"/>
       <geometry>
-        <mesh filename="package://vector_ros/meshes/wheel_rr.stl" scale="0.001 0.001 0.001"/>
+        <mesh filename="package://vector_navigation/meshes/wheel_rr.stl" scale="0.001 0.001 0.001"/>
       </geometry>
       <material name="rubber_black"/>
@@ -115,5 +115,5 @@
       <origin xyz="-0.05 0.02 -0.025" rpy="0 0 0"/>
       <geometry>
-        <mesh filename="package://vector_ros/meshes/lidar_base.stl" scale="0.001 0.001 0.001"/>
+        <mesh filename="package://vector_navigation/meshes/lidar_base.stl" scale="0.001 0.001 0.001"/>
       </geometry>
       <material name="dark_grey"/>
@@ -135,5 +135,5 @@
       <origin xyz="-0.092 -0.0 -0.0732" rpy="0 0 0"/>
       <geometry>
-        <mesh filename="package://vector_ros/meshes/lidar_link.stl" scale="0.001 0.001 0.001"/>
+        <mesh filename="package://vector_navigation/meshes/lidar_link.stl" scale="0.001 0.001 0.001"/>
       </geometry>
       <material name="gunmetal"/>
@@ -155,5 +155,5 @@
       <origin xyz="-0.079875 -0.079 -0.0" rpy="0 0 0"/>
       <geometry>
-        <mesh filename="package://vector_ros/meshes/motor_fl.stl" scale="0.001 0.001 0.001"/>
+        <mesh filename="package://vector_navigation/meshes/motor_fl.stl" scale="0.001 0.001 0.001"/>
       </geometry>
       <material name="dark_grey"/>
@@ -175,5 +175,5 @@
       <origin xyz="0.063825 -0.064 -0.0" rpy="0 0 0"/>
       <geometry>
-        <mesh filename="package://vector_ros/meshes/motor_rl.stl" scale="0.001 0.001 0.001"/>
+        <mesh filename="package://vector_navigation/meshes/motor_rl.stl" scale="0.001 0.001 0.001"/>
       </geometry>
       <material name="dark_grey"/>
@@ -195,5 +195,5 @@
       <origin xyz="-0.079825 0.064 -0.0" rpy="0 0 0"/>
       <geometry>
-        <mesh filename="package://vector_ros/meshes/motor_fr.stl" scale="0.001 0.001 0.001"/>
+        <mesh filename="package://vector_navigation/meshes/motor_fr.stl" scale="0.001 0.001 0.001"/>
       </geometry>
       <material name="dark_grey"/>
@@ -215,5 +215,5 @@
       <origin xyz="-0.071875 -0.089 0.019875" rpy="0 0 0"/>
       <geometry>
-        <mesh filename="package://vector_ros/meshes/wheel_fl.stl" scale="0.001 0.001 0.001"/>
+        <mesh filename="package://vector_navigation/meshes/wheel_fl.stl" scale="0.001 0.001 0.001"/>
       </geometry>
       <material name="rubber_black"/>
@@ -235,5 +235,5 @@
       <origin xyz="0.071776 -0.089 0.019875" rpy="0 0 0"/>
       <geometry>
-        <mesh filename="package://vector_ros/meshes/wheel_rl.stl" scale="0.001 0.001 0.001"/>
+        <mesh filename="package://vector_navigation/meshes/wheel_rl.stl" scale="0.001 0.001 0.001"/>
       </geometry>
       <material name="rubber_black"/>
@@ -255,5 +255,5 @@
       <origin xyz="-0.071776 0.089 0.019875" rpy="0 0 0"/>
       <geometry>
-        <mesh filename="package://vector_ros/meshes/wheel_fr.stl" scale="0.001 0.001 0.001"/>
+        <mesh filename="package://vector_navigation/meshes/wheel_fr.stl" scale="0.001 0.001 0.001"/>
       </geometry>
       <material name="rubber_black"/>
